File: aaXBee.sch (EAGLE design)
At the start: 82 parts, among them Q1 IRLML6244TR, SW1 SW1, SW2 RESET, U1 MCP1640D, U2 MCP1640D, U4 ATmega328P-AU, U5 MCP9808, U6 DS3231, Y1 8MHz

Commit message: As sent to fab.
Parts:
- removed D5: Red, _jc:LEDD0805A
- removed JP5: Run/Pgm, SparkFun:M03LOCK
- removed R17: 249K, _jc:R-US_M0805
- removed SW2: RESET, _jc:SPST-NO-MCTACT-6X3.5-SMT
- removed U6: DS3231, _jc:DS3231
- added D8: Yellow, _jc:LEDD0805A
- added JP4: GNDSEL, SparkFun:M03LOCK
- added R8: 10K, _jc:R-US_M0805
- added SW7: SW7, _jc:SPST-NO-MCTACT-6X3.5-SMT
- added U3: MCP9808, _jc:MCP9808
- B1: value CR2016 -> 2xAA; device _jc:COIN-CELL-2016-SMT -> _jc:BATTERY-2AANOHOLES
- B2: value 2xAA -> CR2016; device _jc:BATTERY-2AANOHOLES -> _jc:COIN-CELL-2016-SMT
- C1, C2, C3, C6, C7: value 10uF -> 100nF
- C10, C11, C8, C9: value 100nF -> 10uF
- C14: value 27pF -> 10uF
- C15: value 27pF -> 100nF
- C4, C5: value 100nF -> 27pF
- D1: value Yellow -> 1N4148; device _jc:LEDD0805A -> _jc:DIODESOD-323F-A
- D2: device _jc:DIODESOD-323F -> _jc:DIODESOD-323F-A
- D3: value 1N4148 -> Red; device _jc:DIODESOD-323F -> _jc:LEDD0805A
- JP3: value GNDSEL -> Run/Pgm
- L1: value 4.7uH -> 10uH; device _jc:INDUCTORNRS4018 -> _jc:INDUCTORM0805
- L2: value 10uH -> 4.7uH; device _jc:INDUCTORM0805 -> _jc:INDUCTORNRS4018
- PR13: value PROTO-3 -> GND
- R1, R3: value 976K -> 10K
- R10: value 2.2K -> 309K
- R11: value 220 -> 249K
- R12: value 10K -> 976K
- R13: value 4.7K -> 562K
- R14: value 1K -> 4.7K
- R16: value 562K -> 1K
- R2: value 309K -> 47.5K
- R4: value 47.5K -> 2.2K
- R5: value 10K -> 2.2K
- R6: value 10K -> 1K
- R7: value 1K -> 220
- R9: value 2.2K -> 976K
- SJ2: value XBee VR Sel -> Reg2 IP; device jumper:SJ2W -> jumper:SJ
- SJ3: value /5V -> XBee VR Sel; device jumper:SJ -> jumper:SJ2W
- SJ4: value 5V -> 3.3V
- SW1: value SW1 -> RESET
- U1: value MCP1640D -> ATmega328P-AU; device _jc:MCP1640 -> atmel:MEGA8-AI
- U2: value MCP1640D -> DS3231; device _jc:MCP1640 -> _jc:DS3231
- U4: value ATmega328P-AU -> MCP1640D; device atmel:MEGA8-AI -> _jc:MCP1640
- U5: value MCP9808 -> MCP1640D; device _jc:MCP9808 -> _jc:MCP1640
- renumbered JP6 to JP1
Connections:
- removed net 32KHZ: U6.32KHZ
- net /RESET: now also C6.1, D1.A, R1.1, SW1.P$1, U1.PC6(/RESET); no longer C5.1, D3.A, R6.1, SW2.P$1, U4.PC6(/RESET)
- net /SS: now also U1.PB2(SS/OC1B); no longer U4.PB2(SS/OC1B)
- net ADC0: now also U1.PC0(ADC0); no longer U4.PC0(ADC0)
- net ADC1: now also U1.PC1(ADC1); no longer U4.PC1(ADC1)
- net ADC2: now also U1.PC2(ADC2); no longer U4.PC2(ADC2)
- net ADC3: now also U1.PC3(ADC3); no longer U4.PC3(ADC3)
- net ADC6: now also C7.2, R3.2, U1.ADC6; no longer C4.2, R5.2, U4.ADC6
- net ADC7: now also C7.1, R2.2, R3.1, U1.ADC7; no longer C4.1, R4.2, R5.1, U4.ADC7
- net AREF: now also C3.1, U1.AREF; no longer C13.1, U4.AREF
- net ASC: now also R16.2; no longer R15.2
- net BAT: now also B1.POS, C8.1, L2.1, R2.1, SJ2.1, U4.VIN; no longer B2.POS, C1.1, L1.1, R4.1, SJ4.1, U1.VIN
- net CTS: now also U1.PD5(T1); no longer U4.PD5(T1)
- net EN: now also U1.PD4(XCK/T0), U4.EN, U5.EN; no longer U1.EN, U2.EN, U4.PD4(XCK/T0)
- net GND: now also B1.NEG, B2.B-, C4.2, C5.2, D3.C, D8.C, JP4.3, R11.2, R13.2, R8.2, SW7.P$2, U1.GND@1, U1.GND@2, U2.NC10, U2.NC11, U2.NC12, U2.NC5, U2.NC6, U2.NC7, U2.NC8, U2.NC9, U3.A0, U3.A1, U3.A2, U3.GND; no longer B1.B-, B2.NEG, C6.2, C7.2, D1.C, D5.C, JP3.3, R12.2, R16.2, R17.2, SW2.P$2, U4.GND@1, U4.GND@2, U5.A0, U5.A1, U5.A2, U6.GND, U6.NC10, U6.NC11, U6.NC12, U6.NC5, U6.NC6, U6.NC7, U6.NC8, U6.NC9
- net INT: now also U1.PD3(INT1), U2./INT-SQW; no longer U4.PD3(INT1), U6./INT-SQW
- net MISO: now also U1.PB4(MISO); no longer U4.PB4(MISO)
- net MOSI: now also U1.PB3(MOSI/OC2); no longer U4.PB3(MOSI/OC2)
- net N$1: now also B2.POS1, U2.VBAT; no longer B1.POS1, U6.VBAT
- net N$12: now also R12.2, R13.1, U5.VFB; no longer R16.1, R3.2, U2.VFB
- net N$13: now also U5.SW; no longer U2.SW
- net N$2: now also D8.A, R6.1; no longer D1.A, R7.1
- net N$24: now also R7.1, R8.1; no longer R11.1, R12.1
- net N$35: now also C10.1, SJ2.2, U5.VIN; no longer C6.1, SJ4.2, U2.VIN
- net N$36: now also JP4.1; no longer JP3.1
- net N$37: now also R14.2, SJ4.1; no longer R13.2, SJ3.1
- net N$38: now also JP3.1; no longer JP5.1
- net N$39: now also C11.1, R12.1, SJ3.1, U5.VOUT; no longer C7.1, R3.1, SJ2.1, U2.VOUT
- net N$41: now also D3.A, R15.1; no longer D5.A, R14.1
- net N$42: now also R16.1; no longer R15.1
- net N$43: now also C4.1, U1.PB6(XTAL1/TOSC1); no longer C14.1, U4.PB6(XTAL1/TOSC1)
- net N$44: now also C5.1, U1.PB7(XTAL2/TOSC2); no longer C15.1, U4.PB7(XTAL2/TOSC2)
- net N$46: now also C2.1, L1.2, U1.AVCC; no longer C12.1, L2.2, U4.AVCC
- net N$6: now also R10.1, R9.2, U4.VFB; no longer R1.2, R2.1, U1.VFB
- net N$7: now also L2.2, U4.SW; no longer L1.2, U1.SW
- net N$8: now also R10.2, R11.1; no longer R17.1, R2.2
- net PB0: now also R6.2, U1.PB0(ICP); no longer R7.2, U4.PB0(ICP)
- net PD7: now also SW7.P$1, U1.PD7(AIN1); no longer SW1.P$1, U4.PD7(AIN1)
- net PPWR: now also C12.1, C13.1, U1.PD2(INT0), U2.VCC, U3.VCC; no longer C11.1, C9.1, U4.PD2(INT0), U5.VCC, U6.VCC
- net RSSI: now also R15.2; no longer R14.2
- net RST: now also C6.2; no longer C5.2
- net RXD: now also JP3.2, U1.PD0(RXD); no longer JP5.2, U4.PD0(RXD)
- net SCK: now also U1.PB5(SCK); no longer U4.PB5(SCK)
- net SCL: now also R5.2, U1.PC5(ADC5/SCL), U2.SCL, U3.SCL; no longer R10.2, U4.PC5(ADC5/SCL), U5.SCL, U6.SCL
- net SDA: now also R4.2, U1.PC4(ADC4/SDA), U2.SDA, U3.SDA; no longer R9.2, U4.PC4(ADC4/SDA), U5.SDA, U6.SDA
- net SGND: now also JP4.2; no longer JP3.2
- net SLP: now also U1.PD6(AIN0); no longer U4.PD6(AIN0)
- net SPWR: now also R7.2, U1.PB1(OC1A); no longer R11.2, U4.PB1(OC1A)
- net TXD: now also SJ4.2, U1.PD1(TXD); no longer SJ3.2, U4.PD1(TXD)
- net VCC: now also C1.1, C9.1, D1.K, L1.1, R1.2, R4.1, R5.1, SJ3.3, U1.VCC@1, U1.VCC@2, U4.VOUT; no longer C2.1, C8.1, D3.K, L2.1, R1.1, R10.1, R6.2, SJ2.3, U1.VOUT, U4.VCC@1, U4.VCC@2
- net XBEE_SUPPLY: now also C14.1, C15.1, R14.1, SJ3.2; no longer C10.1, C3.1, R13.1, SJ2.2
Other:
- note added: "REG1 Main 3.3V or 5V supply"
- note removed: "REG1 Main 5V or 3.3V supply"
- moved on the sheet: C1, C10, C11, C12, C13, C14, C15, C2, C3, C4, C5, C6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
